Commit message: Second commit after changes

File: urdf/youbot.urdf (robot description, URDF)
Before this commit: robot youbot, 11 links, 10 joints
Links:
- added link finger_1, mass 1.0; collision box size=0.1 0.1 0.1; visual cylinder length=0.05 radius=0.005
- link endeff: geometry collision box size=0.1 0.1 0.1; visual cylinder length=0.05 radius=0.05
- link wheel_fl: geometry collision cylinder length=0.076 radius=0.05; visual mesh filename=package://youbot/meshes/mecanum.dae scale=0.002 0.002 0.002
- link wheel_fr: geometry collision cylinder length=0.076 radius=0.05; visual mesh filename=package://youbot/meshes/mecanum.dae scale=0.002 0.002 0.002
- link wheel_rl: geometry collision cylinder length=0.076 radius=0.05; visual mesh filename=package://youbot/meshes/mecanum.dae scale=0.002 0.002 0.002
- link wheel_rr: geometry collision cylinder length=0.076 radius=0.05; visual mesh filename=package://youbot/meshes/mecanum.dae scale=0.002 0.002 0.002
Joints:
- added joint endeff__finger_1: type revolute, parent endeff, child finger_1, origin xyz=0 0 0.05 rpy=0 0 0, axis 0 1 0, limit lower=0 upper=1.57 effort=0 velocity=0
- joint base_link__link_1: limit lower=3.14 upper=-3.14 effort=0 velocity=0 -> lower=0 upper=1.57 effort=0 velocity=0
- joint chassis__base_link: limit lower=3.14 upper=-3.14 effort=0 velocity=0 -> lower=0 upper=1.57 effort=0 velocity=0
- joint chassis__wheel_fl: origin xyz=0.270 -0.200 0 rpy=0 0 0 -> xyz=0.270 -0.230 0 rpy=0 0 0
- joint chassis__wheel_fr: origin xyz=0.270 0.200 0 rpy=0 0 0 -> xyz=0.270 0.230 0 rpy=0 0 0
- joint chassis__wheel_rl: origin xyz=-0.270 -0.200 0 rpy=0 0 0 -> xyz=-0.270 -0.230 0 rpy=0 0 0
- joint chassis__wheel_rr: origin xyz=-0.270 0.200 0 rpy=0 0 0 -> xyz=-0.270 0.230 0 rpy=0 0 0
- joint link_1__link_2: limit lower=3.14 upper=-3.14 effort=0 velocity=0 -> lower=0 upper=1.57 effort=0 velocity=0
- joint link_2__link_3: limit lower=3.14 upper=-3.14 effort=0 velocity=0 -> lower=0 upper=1.57 effort=0 velocity=0
- joint link_3__link_4: limit lower=3.14 upper=-3.14 effort=0 velocity=0 -> lower=0 upper=1.57 effort=0 velocity=0
- joint link_4__endeff: limit lower=3.14 upper=-3.14 effort=0 velocity=0 -> lower=0 upper=1.57 effort=0 velocity=0
